File: Hardware/PCB/Capstone 6-Axis Motor/MotorController.sch (EAGLE design)
At the start: 62 parts, among them CON3 TI-JTAG-CTI-20, J1 768250004CON_768250004_MOL, J10 JUMPER, J2 768250004CON_768250004_MOL, J3 MF-CON-2.54mm-01x03, J4 MF-CON-2.54mm-01x03, J5 MF-CON-2.54mm-01x03, J6 MF-CON-2.54mm-01x03, J7 MF-CON-2.54mm-01x03, J8 JUMPER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

Commit message: Updated PCBs and added custom libraries
Other:
- moved on the sheet: U2
